File: R_Rasmanis_MultiVib/R_Rasmanis_MultiVib.sch (KiCad schematic (older format))
At the start: 21 parts, among them Q1 BC548, Q2 BC548, T1 DMC20601

Commit message: MultiVib
Connections:
- wire segments 68 -> 70
Changed lines of the file:
@@
 EESchema Schematic File Version 4
+LIBS:R_Rasmanis_MultiVib-cache
 EELAYER 26 0
 EELAYER END
@@
 U 1 1 5C809E37
 P 6975 3725
-F 0 "T1" H 7173 3801 31  0000 L CNN
-F 1 "DMC20601" H 7173 3725 50  0000 L CNN
+F 0 "T1" H 6740 3720 31  0000 L CNN
+F 1 "DMC20601" H 6410 3785 50  0000 L CNN
 F 2 "" H 7255 3295 50  0001 C CNN
 F 3 "" H 7255 3295 50  0001 C CNN
@@
 $EndComp
 Wire Wire Line
-	6885 3615 6885 3450
-Wire Wire Line
 	6885 3450 6375 3450
 Wire Wire Line
@@
 Connection ~ 6375 3275
 Wire Wire Line
-	6975 3615 6975 3275
-Wire Wire Line
 	6975 3275 6775 3275
 Connection ~ 6775 3275
 Wire Wire Line
-	5825 4125 6885 4125
-Wire Wire Line
-	6885 4125 6885 3865
-Wire Wire Line
-	7065 3615 7475 3615
-Wire Wire Line
-	7475 3615 7475 3275
-Connection ~ 7475 3275
-Wire Wire Line
-	7065 3865 7230 3865
-Wire Wire Line
-	7230 3865 7230 3475
-Wire Wire Line
 	7230 3475 7125 3475
 Wire Wire Line
@@
 Connection ~ 7125 3275
 Wire Wire Line
-	6975 3865 6975 4125
-Wire Wire Line
-	6975 4125 6885 4125
+	7230 3975 7065 3975
+Wire Wire Line
+	7230 3475 7230 3975
+Wire Wire Line
+	7475 3275 7475 3525
+Connection ~ 7475 3275
+Wire Wire Line
+	7065 3595 7065 3525
+Wire Wire Line
+	7065 3525 7475 3525
+Wire Wire Line
+	7065 3885 7065 3975
+Wire Wire Line
+	6975 4125 6975 3885
+Wire Wire Line
+	5825 4125 6885 4125
+Wire Wire Line
+	6885 3885 6885 4125
 Connection ~ 6885 4125
+Wire Wire Line
+	6885 4125 6975 4125
+Wire Wire Line
+	6885 3595 6885 3450
+Wire Wire Line
+	6975 3275 6975 3595
 $EndSCHEMATC
